File: hardware/kicad_project/hybrid_core_module/midi_vco_module/sequencer_ui.kicad_sch (KiCad schematic)
At the start: 99 parts, among them J11 Conn_01x01_Pin, J12 Conn_01x01_Pin, J13 Conn_01x01_Pin, J14 Conn_01x01_Pin, J15 Conn_01x01_Pin, J16 Conn_01x01_Pin, J17 Conn_01x01_Pin, J18 Conn_01x01_Pin, J19 Conn_01x01_Pin, J20 Conn_01x01_Pin, J21 Conn_01x01_Pin, J22 Conn_01x01_Pin, Q18 2N7002, Q19 2N7002, Q20 2N7002, SW10 RotaryEncoder_Switch_MP, SW11 RotaryEncoder_Switch_MP, SW9 SW_Rotary_1x4_MP, U15 MCP23008-xSO, U25 MCP23017_SO

Commit message: components placement (interface) components placement per section
Parts:
- D16, D17, D18, D19, D20, D21, D22, D23, D24, D25, D26, D27, D28, D29, D30, D31: footprint mylib:LED-3528 -> LED_THT:LED_D3.0mm_Clear; Manufacturer SONGXIN LIGHT -> Shenzhen xiangbang; Manufacturer PartNumer SX-3528-AMBER-ORANGE -> ORANGE LED 3MM
- RV13: footprint Potentiometer_THT:Potentiometer_Bourns_3296W_Vertical -> mylib:Potentiometer_RV09_Single_Vertical
Changed lines of the file:
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@@
 			)
 		)
-		(property "Footprint" "mylib:LED-3528"
+		(property "Footprint" "LED_THT:LED_D3.0mm_Clear"
 			(at 160.02 27.94 0)
 			(effects
@@
 			)
 		)
-		(property "Manufacturer" "SONGXIN LIGHT"
+		(property "Manufacturer" "Shenzhen xiangbang "
 			(at 160.02 27.94 90)
 			(effects
@@
 			)
 		)
-		(property "Manufacturer PartNumer" "SX-3528-AMBER-ORANGE "
+		(property "Manufacturer PartNumer" "ORANGE  LED 3MM"
 			(at 160.02 27.94 90)
 			(effects
@@
 			)
 		)
-		(property "Footprint" "mylib:LED-3528"
+		(property "Footprint" "LED_THT:LED_D3.0mm_Clear"
 			(at 186.69 27.94 0)
 			(effects
@@
 			)
 		)
-		(property "Manufacturer" "SONGXIN LIGHT"
+		(property "Manufacturer" "Shenzhen xiangbang "
 			(at 186.69 27.94 90)
 			(effects
@@
 			)
 		)
-		(property "Manufacturer PartNumer" "SX-3528-AMBER-ORANGE "
+		(property "Manufacturer PartNumer" "ORANGE  LED 3MM"
 			(at 186.69 27.94 90)
 			(effects
@@
 			)
 		)
-		(property "Footprint" "Potentiometer_THT:Potentiometer_Bourns_3296W_Vertical"
+		(property "Footprint" "mylib:Potentiometer_RV09_Single_Vertical"
 			(at 50.8 180.34 0)
 			(effects
@@
 			)
 		)
-		(property "Footprint" "mylib:LED-3528"
+		(property "Footprint" "LED_THT:LED_D3.0mm_Clear"
 			(at 204.47 49.53 0)
 			(effects
@@
 			)
 		)
-		(property "Manufacturer" "SONGXIN LIGHT"
+		(property "Manufacturer" "Shenzhen xiangbang "
 			(at 204.47 49.53 90)
 			(effects
@@
 			)
 		)
-		(property "Manufacturer PartNumer" "SX-3528-AMBER-ORANGE "
+		(property "Manufacturer PartNumer" "ORANGE  LED 3MM"
 			(at 204.47 49.53 90)
 			(effects
@@
 			)
 		)
-		(property "Footprint" "mylib:LED-3528"
+		(property "Footprint" "LED_THT:LED_D3.0mm_Clear"
 			(at 204.47 27.94 0)
 			(effects
@@
 			)
 		)
-		(property "Manufacturer" "SONGXIN LIGHT"
+		(property "Manufacturer" "Shenzhen xiangbang "
 			(at 204.47 27.94 90)
 			(effects
@@
 			)
 		)
-		(property "Manufacturer PartNumer" "SX-3528-AMBER-ORANGE "
+		(property "Manufacturer PartNumer" "ORANGE  LED 3MM"
 			(at 204.47 27.94 90)
 			(effects
@@
 			)
 		)
-		(property "Footprint" "mylib:LED-3528"
+		(property "Footprint" "LED_THT:LED_D3.0mm_Clear"
 			(at 195.58 27.94 0)
 			(effects
@@
 			)
 		)
-		(property "Manufacturer" "SONGXIN LIGHT"
+		(property "Manufacturer" "Shenzhen xiangbang "
 			(at 195.58 27.94 90)
 			(effects
@@
 			)
 		)
-		(property "Manufacturer PartNumer" "SX-3528-AMBER-ORANGE "
+		(property "Manufacturer PartNumer" "ORANGE  LED 3MM"
 			(at 195.58 27.94 90)
 			(effects
@@
 			)
 		)
-		(property "Footprint" "mylib:LED-3528"
+		(property "Footprint" "LED_THT:LED_D3.0mm_Clear"
 			(at 142.24 27.94 0)
 			(effects
@@
 			)
 		)
-		(property "Manufacturer" "SONGXIN LIGHT"
+		(property "Manufacturer" "Shenzhen xiangbang "
 			(at 142.24 27.94 90)
 			(effects
@@
 			)
 		)
-		(property "Manufacturer PartNumer" "SX-3528-AMBER-ORANGE "
+		(property "Manufacturer PartNumer" "ORANGE  LED 3MM"
 			(at 142.24 27.94 90)
 			(effects
@@
 			)
 		)
-		(property "Footprint" "mylib:LED-3528"
+		(property "Footprint" "LED_THT:LED_D3.0mm_Clear"
 			(at 168.91 49.53 0)
 			(effects
@@
 			)
 		)
-		(property "Manufacturer" "SONGXIN LIGHT"
+		(property "Manufacturer" "Shenzhen xiangbang "
 			(at 168.91 49.53 90)
 			(effects
@@
 			)
 		)
-		(property "Manufacturer PartNumer" "SX-3528-AMBER-ORANGE "
+		(property "Manufacturer PartNumer" "ORANGE  LED 3MM"
 			(at 168.91 49.53 90)
 			(effects
@@
 			)
 		)
-		(property "Footprint" "mylib:LED-3528"
+		(property "Footprint" "LED_THT:LED_D3.0mm_Clear"
 			(at 151.13 27.94 0)
 			(effects
@@
 			)
 		)
-		(property "Manufacturer" "SONGXIN LIGHT"
+		(property "Manufacturer" "Shenzhen xiangbang "
 			(at 151.13 27.94 90)
 			(effects
@@
 			)
 		)
-		(property "Manufacturer PartNumer" "SX-3528-AMBER-ORANGE "
+		(property "Manufacturer PartNumer" "ORANGE  LED 3MM"
 			(at 151.13 27.94 90)
 			(effects
@@
 			)
 		)
-		(property "Footprint" "mylib:LED-3528"
+		(property "Footprint" "LED_THT:LED_D3.0mm_Clear"
 			(at 195.58 49.53 0)
 			(effects
@@
 			)
 		)
-		(property "Manufacturer" "SONGXIN LIGHT"
+		(property "Manufacturer" "Shenzhen xiangbang "
 			(at 195.58 49.53 90)
 			(effects
@@
 			)
 		)
-		(property "Manufacturer PartNumer" "SX-3528-AMBER-ORANGE "
+		(property "Manufacturer PartNumer" "ORANGE  LED 3MM"
 			(at 195.58 49.53 90)
 			(effects
@@
 			)
 		)
-		(property "Footprint" "mylib:LED-3528"
+		(property "Footprint" "LED_THT:LED_D3.0mm_Clear"
 			(at 177.8 27.94 0)
 			(effects
@@
 			)
 		)
-		(property "Manufacturer" "SONGXIN LIGHT"
+		(property "Manufacturer" "Shenzhen xiangbang "
 			(at 177.8 27.94 90)
 			(effects
@@
 			)
 		)
-		(property "Manufacturer PartNumer" "SX-3528-AMBER-ORANGE "
+		(property "Manufacturer PartNumer" "ORANGE  LED 3MM"
 			(at 177.8 27.94 90)
 			(effects
@@
 			)
 		)
-		(property "Footprint" "mylib:LED-3528"
+		(property "Footprint" "LED_THT:LED_D3.0mm_Clear"
 			(at 168.91 27.94 0)
 			(effects
@@
 			)
 		)
-		(property "Manufacturer" "SONGXIN LIGHT"
+		(property "Manufacturer" "Shenzhen xiangbang "
 			(at 168.91 27.94 90)
 			(effects
@@
 			)
 		)
-		(property "Manufacturer PartNumer" "SX-3528-AMBER-ORANGE "
+		(property "Manufacturer PartNumer" "ORANGE  LED 3MM"
 			(at 168.91 27.94 90)
 			(effects
@@
 			)
 		)
-		(property "Footprint" "mylib:LED-3528"
+		(property "Footprint" "LED_THT:LED_D3.0mm_Clear"
 			(at 142.24 49.53 0)
 			(effects
@@
 			)
 		)
-		(property "Manufacturer" "SONGXIN LIGHT"
+		(property "Manufacturer" "Shenzhen xiangbang "
 			(at 142.24 49.53 90)
 			(effects
@@
 			)
 		)
-		(property "Manufacturer PartNumer" "SX-3528-AMBER-ORANGE "
+		(property "Manufacturer PartNumer" "ORANGE  LED 3MM"
 			(at 142.24 49.53 90)
 			(effects
@@
 			)
 		)
-		(property "Footprint" "mylib:LED-3528"
+		(property "Footprint" "LED_THT:LED_D3.0mm_Clear"
 			(at 177.8 49.53 0)
 			(effects
@@
 			)
 		)
-		(property "Manufacturer" "SONGXIN LIGHT"
+		(property "Manufacturer" "Shenzhen xiangbang "
 			(at 177.8 49.53 90)
 			(effects
@@
 			)
 		)
-		(property "Manufacturer PartNumer" "SX-3528-AMBER-ORANGE "
+		(property "Manufacturer PartNumer" "ORANGE  LED 3MM"
 			(at 177.8 49.53 90)
 			(effects
@@
 			)
 		)
-		(property "Footprint" "mylib:LED-3528"
+		(property "Footprint" "LED_THT:LED_D3.0mm_Clear"
 			(at 160.02 49.53 0)
 			(effects
@@
 			)
 		)
-		(property "Manufacturer" "SONGXIN LIGHT"
+		(property "Manufacturer" "Shenzhen xiangbang "
 			(at 160.02 49.53 90)
 			(effects
@@
 			)
 		)
-		(property "Manufacturer PartNumer" "SX-3528-AMBER-ORANGE "
+		(property "Manufacturer PartNumer" "ORANGE  LED 3MM"
 			(at 160.02 49.53 90)
 			(effects
@@
 			)
 		)
-		(property "Footprint" "mylib:LED-3528"
+		(property "Footprint" "LED_THT:LED_D3.0mm_Clear"
 			(at 151.13 49.53 0)
 			(effects
@@
 			)
 		)
-		(property "Manufacturer" "SONGXIN LIGHT"
+		(property "Manufacturer" "Shenzhen xiangbang "
 			(at 151.13 49.53 90)
 			(effects
@@
 			)
 		)
-		(property "Manufacturer PartNumer" "SX-3528-AMBER-ORANGE "
+		(property "Manufacturer PartNumer" "ORANGE  LED 3MM"
 			(at 151.13 49.53 90)
 			(effects
@@
 			)
 		)
-		(property "Footprint" "mylib:LED-3528"
+		(property "Footprint" "LED_THT:LED_D3.0mm_Clear"
 			(at 186.69 49.53 0)
 			(effects
@@
 			)
 		)
-		(property "Manufacturer" "SONGXIN LIGHT"
+		(property "Manufacturer" "Shenzhen xiangbang "
 			(at 186.69 49.53 90)
 			(effects
@@
 			)
 		)
-		(property "Manufacturer PartNumer" "SX-3528-AMBER-ORANGE "
+		(property "Manufacturer PartNumer" "ORANGE  LED 3MM"
 			(at 186.69 49.53 90)
 			(effects

Commit message: - placement done - routing 60%
Parts:
- removed R196: 100R, Resistor_SMD:R_0402_1005Metric, symbol Device:R
- added C105: 1nF, Capacitor_SMD:C_0402_1005Metric, symbol Device:C
- R113: value 1k -> 100R; Manufacturer PartNumer RT0402FRE071KL -> RT0402FRE07100RL
- SW10, SW11: footprint Rotary_Encoder:RotaryEncoder_Alps_EC11E-Switch_Vertical_H20mm -> mylib:RotaryEncoder_Alps_EC11E-Switch_Vertical_H20mm_CircularMountingHoles
Connections:
- net BT_REC_OUT: now also U15.16 (GP6); no longer U15.14 (GP4)
- net BT_START_LED: now also U15.15 (GP5); no longer U15.16 (GP6)
- net BT_START_OUT: now also U15.14 (GP4); no longer U15.13 (GP3)
- net BT_STOP_LED: now also U15.13 (GP3); no longer U15.15 (GP5)
- net GATE_LENGTH_OUT: now also R139.1, C105.2; no longer RV13.2
- net GND: now also C105.1
- net LED1: now also U25.1 (GPB0); no longer U25.21 (GPA0)
- net LED10: now also U25.27 (GPA6); no longer U25.2 (GPB1)
- net LED11: now also U25.26 (GPA5); no longer U25.3 (GPB2)
- net LED12: now also U25.25 (GPA4); no longer U25.4 (GPB3)
- net LED13: now also U25.24 (GPA3); no longer U25.5 (GPB4)
- net LED14: now also U25.23 (GPA2); no longer U25.6 (GPB5)
- net LED15: now also U25.22 (GPA1); no longer U25.7 (GPB6)
- net LED16: now also U25.21 (GPA0); no longer U25.8 (GPB7)
- net LED2: now also U25.2 (GPB1); no longer U25.22 (GPA1)
- net LED3: now also U25.3 (GPB2); no longer U25.23 (GPA2)
- net LED4: now also U25.4 (GPB3); no longer U25.24 (GPA3)
- net LED5: now also U25.5 (GPB4); no longer U25.25 (GPA4)
- net LED6: now also U25.6 (GPB5); no longer U25.26 (GPA5)
- net LED7: now also U25.7 (GPB6); no longer U25.27 (GPA6)
- net LED8: now also U25.8 (GPB7); no longer U25.28 (GPA7)
- net LED9: now also U25.28 (GPA7); no longer U25.1 (GPB0)
- net SEQ_CLK_SW: now also R189.1, SW10.S1
- net SEQ_STEPS_SW: now also R138.1, SW11.S1; no longer R139.2
- new net: R139.2, RV13.2
Other:
- moved on the sheet: RV13
