File: hardware/kicad_project/hybrid_core_module/midi_vco_module/midi_vco_module.kicad_pcb (KiCad board)
At the start: 2 copper layers, 152.4 x 111 mm, 474 parts, among them J1 AudioJack2_SwitchT, J10 Conn_01x06_Pin, J11 Conn_01x01_Pin, J12 Conn_01x01_Pin, J13 Conn_01x01_Pin, J14 Conn_01x01_Pin, J15 Conn_01x01_Pin, J16 Conn_01x01_Pin, J17 Conn_01x01_Pin, J18 Conn_01x01_Pin, J19 Conn_01x01_Pin, J2 Screw_Terminal_01x08, J20 Conn_01x01_Pin, J21 Conn_01x01_Pin, J22 Conn_01x01_Pin, J23 Conn_01x03_Pin, J3 AudioJack2_SwitchT, J4 AudioJack2_SwitchT, J5 AudioJack2_SwitchT, J6 AudioJack2_SwitchT, J7 Conn_02x03_Odd_Even, J8 AudioJack2_SwitchT, J9 Conn_02x08_Odd_Even, Q1 2N7002, Q10 2N7002, Q11 BCM847BS, Q12 SSM2212, Q13 2N7002, Q13 BC848, Q14 BF545A, Q15 2N7002, Q16 2N7002, Q17 BCM847BS, Q18 2N7002, Q19 2N7002, Q2 BC848, Q20 2N7002, Q3 BC848, Q4 2N7002, Q5 BSS83P, Q6 SSM2212, Q7 2N7002, Q7 BC848, Q8 BF545A, Q9 2N7002, SW10 RotaryEncoder_Switch_MP, SW11 RotaryEncoder_Switch_MP, SW2 SW_Rotary_1x4_MP, SW3 SW_Rotary_1x4_MP, SW4 SW_Push, SW5 SW_Push, SW6 SW_SPDT, SW9 SW_Rotary_1x4_MP, U1 SHT4x, U10 CP2102N-Axx-xQFN28, U11 TL074, U12 LM311DR, U13 TL072, U14 TL074, U15 MCP23008-xSO, U16 MC79M12CDTRKG, U17 SHT4x, U18 LM4040DBZ-2.5, U19 MCP4922-ESL, U2 TL071, U21 TL074, U22 LM311DR, U23 TL072, U24 TL074, U25 MCP23017_SO, U3 USBLC6-2SC6, U4 TPS65131TRGERQ1, U5 MC78M12CDTRKG, U7 6N137, U8 AZ1117CH2-3.3, U9 ESP32-WROOM-32E

Commit message: - placement done - routing 60%
Parts:
- removed the Q13 at (413.1, -32.3)
- removed the Q13 at (395.1, -26.0)
- removed the Q7 at (395.1, -30.6)
- removed the Q7 at (419.4, -36.9)
- removed R196: 100R, Resistor_SMD:R_0402_1005Metric
- removed U3: USBLC6-2SC6, Package_TO_SOT_SMD:SOT-23-6
- added C100: 100nF, Capacitor_SMD:C_0402_1005Metric, F.Cu at (51.2, 83.3)
- added C101: 100nF, Capacitor_SMD:C_0402_1005Metric, F.Cu at (110.2, 77.8)
- added C102: 1uF, Capacitor_SMD:C_0805_2012Metric, F.Cu at (98.2, 84.3)
- added C103: 1uF, Capacitor_SMD:C_0805_2012Metric, F.Cu at (106.2, 77.3)
- added C104: 100nF, Capacitor_SMD:C_0402_1005Metric, F.Cu at (95.5, 84.5)
- added C105: 1nF, Capacitor_SMD:C_0402_1005Metric, F.Cu at (111.3, 48.9)
- added C97: 100nF, Capacitor_SMD:C_0402_1005Metric, F.Cu at (61.0, 78.0)
- added C98: 1uF, Capacitor_SMD:C_0805_2012Metric, F.Cu at (54.2, 84.8)
- added C99: 1uF, Capacitor_SMD:C_0805_2012Metric, F.Cu at (60.2, 75.8)
- added D35: ESD9B5.0ST5G, Diode_SMD:D_SOD-923, F.Cu at (38.8, 123.8)
- added D36: ESD9B5.0ST5G, Diode_SMD:D_SOD-923, F.Cu at (36.2, 123.8)
- added D37: ESD9B5.0ST5G, Diode_SMD:D_SOD-923, F.Cu at (28.0, 123.8)
- added Q13: 2N7002, Package_TO_SOT_SMD:SOT-23, F.Cu at (85.2, 101.8)
- added Q7: 2N7002, Package_TO_SOT_SMD:SOT-23, F.Cu at (94.8, 102.3)
- added R211: 820k, Resistor_SMD:R_0402_1005Metric, F.Cu at (50.2, 91.8)
- added R212: 820k, Resistor_SMD:R_0402_1005Metric, F.Cu at (85.2, 85.8)
- R113: value 1k -> 100R
- R202, R205: value 10k -> 5.1M
- SW10, SW11: footprint Rotary_Encoder:RotaryEncoder_Alps_EC11E-Switch_Vertical_H20mm -> mylib:RotaryEncoder_Alps_EC11E-Switch_Vertical_H20mm_CircularMountingHoles
- U7: footprint Package_DIP:PowerIntegrations_SMD-8 -> Package_DIP:DIP-8_W7.62mm
- moved C50 566.4 mm to (99.2, 57.3), turned to 90 degrees
- moved R158 562.3 mm to (38.2, 84.8)
- moved C71 559.7 mm to (47.2, 95.3), turned to -90 degrees
- moved C48 559.5 mm to (100.8, 57.8), turned to 90 degrees
- moved R156 557.8 mm to (40.2, 84.8), turned to 180 degrees
- moved C69 557.4 mm to (48.8, 94.8), turned to -90 degrees
- moved C49 555.4 mm to (110.2, 56.3), turned to 90 degrees
- moved TP24 554.7 mm to (54.2, 63.3)
- moved TP23 552.9 mm to (56.8, 75.3)
- moved R164 552.3 mm to (54.2, 64.8)
- moved U13 552.1 mm to (46.8, 87.8), turned to -90 degrees
- moved U21 551.7 mm to (105.3, 58.5)
- moved TP21 550.9 mm to (44.2, 94.3), turned to -90 degrees
- moved R59 550.7 mm to (98.8, 50.8), turned to 0 degrees
- moved R62 550.7 mm to (98.8, 51.8), turned to 180 degrees
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Connections:
- net Net-(D4-A) renamed /POWER_AND_INPUTS/INP
- net Net-(D8-K) renamed /POWER_AND_INPUTS/OUTN
- J10 pad 4: Net-(J10-Pin_4) -> /MCU/CP_D_N
- J10 pad 5: Net-(J10-Pin_5) -> /MCU/CP_D_P
- R138 pad 1: Net-(R138-Pad1) -> /SEQUENCER_UI/SEQ_STEPS_SW
- R139 pad 1: Net-(R138-Pad1) -> /MCU/SEQ_GATE_LENGTH_IN
- R139 pad 2: /SEQUENCER_UI/SEQ_STEPS_SW -> Net-(R139-Pad2)
- R189 pad 1: Net-(R189-Pad1) -> /SEQUENCER_UI/SEQ_CLK_SW
- R202 pad 1: Net-(Q7-B) -> +12V
- R202 pad 2: /CALIBATION_MODE -> Net-(R202-Pad2)
- R205 pad 1: Net-(Q13-B) -> +12V
- R205 pad 2: /CALIBATION_MODE -> Net-(R205-Pad2)
- RV13 pad 2: /MCU/SEQ_GATE_LENGTH_IN -> Net-(R139-Pad2)
- RV17 pad 1: +12V -> Net-(R202-Pad2)
- RV17 pad 3: GND -> Net-(R211-Pad1)
- RV4 pad 1: +12V -> Net-(R205-Pad2)
- RV4 pad 3: GND -> Net-(R212-Pad1)
- SW10 pad S1: Net-(R189-Pad1) -> /SEQUENCER_UI/SEQ_CLK_SW
- SW11 pad S1: Net-(R138-Pad1) -> /SEQUENCER_UI/SEQ_STEPS_SW
- U10 pad 4: /MCU/CP_DP -> /MCU/CP_D_P
- U10 pad 5: /MCU/CP_DN -> /MCU/CP_D_N
- U15 pad 13: /SEQUENCER_UI/BT_START_OUT -> /SEQUENCER_UI/BT_STOP_LED
- U15 pad 14: /SEQUENCER_UI/BT_REC_OUT -> /SEQUENCER_UI/BT_START_OUT
- U15 pad 15: /SEQUENCER_UI/BT_STOP_LED -> /SEQUENCER_UI/BT_START_LED
- U15 pad 16: /SEQUENCER_UI/BT_START_LED -> /SEQUENCER_UI/BT_REC_OUT
- U25 pad 1: /SEQUENCER_UI/LED9 -> /SEQUENCER_UI/LED1
- U25 pad 2: /SEQUENCER_UI/LED10 -> /SEQUENCER_UI/LED2
- U25 pad 21: /SEQUENCER_UI/LED1 -> /SEQUENCER_UI/LED16
- U25 pad 22: /SEQUENCER_UI/LED2 -> /SEQUENCER_UI/LED15
- U25 pad 23: /SEQUENCER_UI/LED3 -> /SEQUENCER_UI/LED14
- U25 pad 24: /SEQUENCER_UI/LED4 -> /SEQUENCER_UI/LED13
- U25 pad 25: /SEQUENCER_UI/LED5 -> /SEQUENCER_UI/LED12
- U25 pad 26: /SEQUENCER_UI/LED6 -> /SEQUENCER_UI/LED11
- U25 pad 27: /SEQUENCER_UI/LED7 -> /SEQUENCER_UI/LED10
- U25 pad 28: /SEQUENCER_UI/LED8 -> /SEQUENCER_UI/LED9
- U25 pad 3: /SEQUENCER_UI/LED11 -> /SEQUENCER_UI/LED3
- U25 pad 4: /SEQUENCER_UI/LED12 -> /SEQUENCER_UI/LED4
- U25 pad 5: /SEQUENCER_UI/LED13 -> /SEQUENCER_UI/LED5
- U25 pad 6: /SEQUENCER_UI/LED14 -> /SEQUENCER_UI/LED6
- U25 pad 7: /SEQUENCER_UI/LED15 -> /SEQUENCER_UI/LED7
- U25 pad 8: /SEQUENCER_UI/LED16 -> /SEQUENCER_UI/LED8
Routing:
- net /MCU/I2C_SCL: track 0.00 -> 141.0 mm, vias 0 -> 3
- net /MCU/I2C_SDA: track 0.00 -> 138.2 mm, vias 0 -> 3
- net VUSB1: track 0.00 -> 111.4 mm
- net Net-(J11-Pin_1): track 0.00 -> 93.6 mm
- net /SAW_PULSE_A/V_PWM_CTRL: track 0.00 -> 83.6 mm
- net Net-(J17-Pin_1): track 0.00 -> 78.8 mm
- net Net-(J20-Pin_1): track 0.00 -> 77.4 mm
- net Net-(J22-Pin_1): track 0.00 -> 75.3 mm
- net Net-(J13-Pin_1): track 0.00 -> 72.0 mm
- net Net-(Q11A-C1): track 0.00 -> 67.7 mm
- net /VCO_SAW_B/V_PITCHSHIFT: track 0.00 -> 63.3 mm, vias 0 -> 2
- net Net-(J15-Pin_1): track 0.00 -> 62.4 mm
- net /SAW_PULSE_B/V_SAW: track 0.00 -> 58.1 mm
- net Net-(D25-K): track 0.00 -> 56.1 mm, vias 0 -> 1
- net Net-(D17-K): track 0.00 -> 54.9 mm, vias 0 -> 1
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- added copper zone on F.Cu, net /POWER_AND_INPUTS/OUTN
Other:
- outline, holes or cut-outs redrawn
- copper layers 2 -> 4
- board text added: "- 0 +"
- board text added: "KEEPOUT"
- board text removed: "Osc2 Wave Out"

Commit message: routing continued.
Parts:
- moved D10 43.3 mm to (112.4, 85.8)
- moved D9 38.9 mm to (114.0, 95.0), turned to -90 degrees
- moved J2 34.3 mm to (172.6, 77.4), turned to -90 degrees
- moved TP4 13.4 mm to (107.5, 101.0)
- moved C11 11.3 mm to (103.0, 117.0)
- moved C12 11.3 mm to (105.0, 117.0)
- moved C9 7.44 mm to (101.0, 122.0), turned to 90 degrees
- moved R141 5.94 mm to (35.2, 42.2), turned to 90 degrees
- moved R7 5.71 mm to (114.7, 119.0)
- moved C14 5.54 mm to (115.0, 116.5)
- moved TP19 5.47 mm to (52.5, 61.0)
- moved TP32 5.24 mm to (124.0, 104.5)
- moved R140 5.17 mm to (35.2, 39.6), turned to 90 degrees
- moved C13 4.82 mm to (110.4, 99.0), turned to -90 degrees
- moved R58 4.71 mm to (54.9, 55.3), turned to 180 degrees
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Connections:
- J2 pad 3: /VELOCITY_OUT_INTER -> /GATE_OUT_INTER
- J2 pad 4: /GATE_OUT_INTER -> /VELOCITY_OUT_INTER
Routing:
- net /OSC2_OUT_INTER: track 0.00 -> 205.8 mm
- net /OSC1_OUT_INTER: track 0.00 -> 173.5 mm
- net /OSC_LFO_INTER: track 0.00 -> 169.7 mm, vias 0 -> 1
- net /GATE_OUT_INTER: track 0.00 -> 117.2 mm
- net /MCU/SEQ_STEPS_A: track 3.28 -> 118.9 mm, vias 0 -> 2
- net Net-(R139-Pad2): track 14.8 -> 129.2 mm, vias 1 -> 2
- net /VELOCITY_OUT_INTER: track 0.00 -> 112.8 mm
- net /MCU/SEQ_CLK_A: track 1.01 -> 110.3 mm, vias 0 -> 2
- net /MCU/SEQ_STEPS_B: track 4.82 -> 108.6 mm, vias 0 -> 2
- net /MCU/SEQ_CLK_B: track 3.71 -> 92.6 mm, vias 0 -> 2
- net Net-(R113-Pad2): track 12.8 -> 100.6 mm, vias 1 -> 2
- net /SYNTH_CV/CTRL_VELOCITY_OUT: track 2.98 -> 77.4 mm
- net /MCU/OSC1_FB: track 2.98 -> 75.7 mm, vias 0 -> 2
- net /MCU/MCP2_INT: track 4.34 -> 73.9 mm, vias 0 -> 2
- net Net-(U11A-+): track 0.00 -> 67.8 mm, vias 0 -> 2
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- added copper zone on F.Cu, net /POWER_AND_INPUTS/INP
